File: keyhalld.kicad_pcb (KiCad board)
At the start: 4 copper layers, 89 parts, among them J1 Conn_ARM_SWD_TagConnect_TC203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, J2 USB_C_Receptacle_USB2.0_16P, SW1 HallSwitch, SW10 HallSwitch, SW11 HallSwitch, SW12 HallSwitch, SW13 HallSwitch, SW14 HallSwitch, SW15 HallSwitch, SW16 HallSwitch, SW17 HallSwitch, SW18 HallSwitch, SW2 HallSwitch, SW3 HallSwitch, SW4 HallSwitch, SW5 HallSwitch, SW6 HallSwitch, SW7 HallSwitch, SW8 HallSwitch, SW9 HallSwitch, U1 AMS1117-3.3, U10 DRV5055A4xDBZxQ1, U11 DRV5055A4xDBZxQ1, U12 DRV5055A4xDBZxQ1, U13 DRV5055A4xDBZxQ1, U14 DRV5055A4xDBZxQ1, U15 DRV5055A4xDBZxQ1, U16 DRV5055A4xDBZxQ1, U17 DRV5055A4xDBZxQ1, U18 DRV5055A4xDBZxQ1, U19 DRV5055A4xDBZxQ1, U2 USBLC6-2SC6, U20 DRV5055A4xDBZxQ1, U21 DRV5055A4xDBZxQ1, U22 DRV5055A4xDBZxQ1, U3 RP2350A, U4 CD74HC4067M, U5 DRV5055A4xDBZxQ1, U6 DRV5055A4xDBZxQ1, U7 DRV5055A4xDBZxQ1, U8 DRV5055A4xDBZxQ1, U9 DRV5055A4xDBZxQ1, Y1 12MHz

Commit message: add connector footprint; mounting holes; reannotate
Parts:
- added C12: 100n, Capacitor_SMD:C_0603_1608Metric_Pad1.08x0.95mm_HandSolder, F.Cu at (107.0, 94.7)
- added H1: MountingHole_Pad, MountingHole:MountingHole_2.2mm_M2, F.Cu at (109.0, 105.0)
- added H2: MountingHole_Pad, MountingHole:MountingHole_2.2mm_M2, F.Cu at (109.0, 110.9)
- added H3: MountingHole_Pad, MountingHole:MountingHole_2.2mm_M2, F.Cu at (109.0, 116.9)
- added H4: MountingHole_Pad, MountingHole:MountingHole_2.2mm_M2, F.Cu at (109.0, 122.8)
- added J3: Conn_01x05_Pin, Connector_PinHeader_1.00mm:PinHeader_1x05_P1.00mm_Horizontal, F.Cu at (113.5, 94.5)
- added R9: 1.5K, Resistor_SMD:R_0603_1608Metric_Pad0.98x0.95mm_HandSolder, F.Cu at (107.0, 92.2)
- renumbered C12 to C13, C13 to C14, C14 to C15, C15 to C16, C16 to C17, C17 to C18, C18 to C19, C19 to C20, C20 to C21, C21 to C22, C22 to C23, C23 to C24, C24 to C25, C25 to C26, C26 to C27, C27 to C28, C28 to C29, C29 to C30, C30 to C31, C31 to C32, C32 to C33, C33 to C34, C34 to C35, C35 to C36, C36 to C37, R9 to R10
Connections:
- U4 pad 12: unconnected-(U4-GND-Pad12) -> GND
