File: keyhalld.kicad_sch (KiCad schematic)
At the start: 36 parts, among them J1 Conn_ARM_SWD_TagConnect_TC203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, J2 USB_C_Receptacle_USB2.0_16P, J3 Conn_01x05_Pin, U1 AMS1117-3.3, U2 USBLC6-2SC6, U3 RP2350A, U4 CD74HC4067M, Y1 12MHz

Commit message: update schematic; add portal to heaven;
Parts:
- added C12: 100n, Capacitor_SMD:C_0603_1608Metric_Pad1.08x0.95mm_HandSolder, symbol Device:C
- added R?: 1.5K, Resistor_SMD:R_0603_1608Metric_Pad0.98x0.95mm_HandSolder, symbol Device:R
- renumbered C12 to C13, C13 to C14, C14 to C15, C15 to C16, C16 to C17, C17 to C18, C18 to C19
Connections:
- net +3.3V: now also R?.2
- net GND: now also U4.12 (GND), C12.1
- net RUN: now also C12.2, R?.1
- no-connect marks 27 -> 29
Other:
- note added: "Pad Connector for IDC-2050 cable"

Commit message: add connector footprint; mounting holes; reannotate
Parts:
- added H1, H2, H3, H4: MountingHole_Pad, MountingHole:MountingHole_2.2mm_M2, symbol Mechanical:MountingHole_Pad
- J3: footprint (none) -> Connector_PinHeader_1.00mm:PinHeader_1x05_P1.00mm_Horizontal
- gave numbers to parts that had none: 1
- renumbered R9 to R10
Connections:
- net GND: now also H1.1, H2.1, H3.1, H4.1
