File: hallswitches.kicad_sch (KiCad schematic)
At the start: 54 parts, among them SW1 HallSwitch, SW10 HallSwitch, SW11 HallSwitch, SW12 HallSwitch, SW13 HallSwitch, SW14 HallSwitch, SW15 HallSwitch, SW16 HallSwitch, SW17 HallSwitch, SW18 HallSwitch, SW2 HallSwitch, SW3 HallSwitch, SW4 HallSwitch, SW5 HallSwitch, SW6 HallSwitch, SW7 HallSwitch, SW8 HallSwitch, SW9 HallSwitch, U10 DRV5055A4xDBZxQ1, U11 DRV5055A4xDBZxQ1, U12 DRV5055A4xDBZxQ1, U13 DRV5055A4xDBZxQ1, U14 DRV5055A4xDBZxQ1, U15 DRV5055A4xDBZxQ1, U16 DRV5055A4xDBZxQ1, U17 DRV5055A4xDBZxQ1, U18 DRV5055A4xDBZxQ1, U19 DRV5055A4xDBZxQ1, U20 DRV5055A4xDBZxQ1, U21 DRV5055A4xDBZxQ1, U22 DRV5055A4xDBZxQ1, U5 DRV5055A4xDBZxQ1, U6 DRV5055A4xDBZxQ1, U7 DRV5055A4xDBZxQ1, U8 DRV5055A4xDBZxQ1, U9 DRV5055A4xDBZxQ1

Commit message: update schematic; add portal to heaven;
Parts:
- renumbered C19 to C20, C20 to C21, C21 to C22, C22 to C23, C23 to C24, C24 to C25, C25 to C26, C26 to C27, C27 to C28, C28 to C29, C29 to C30, C30 to C31, C31 to C32, C32 to C33, C33 to C34, C34 to C35, C35 to C36, C36 to C37

Commit message: Modularize sheets. Still WIP
Connections:
- net GND renamed GNDA

Commit message: Modified Power supplies, lost some sanity
Parts:
- renumbered C25 to C10, C26 to C11, C27 to C12, C28 to C13, C29 to C14, C30 to C15, C31 to C16, C32 to C17, C33 to C18, C34 to C19, C35 to C20, C36 to C21, C37 to C22, C20 to C5, C21 to C6, C22 to C7, C23 to C8, C24 to C9, U12 to U10, U13 to U11, U14 to U12, U15 to U13, U16 to U14, U17 to U15, U18 to U16, U19 to U17, U20 to U18, U21 to U19, U22 to U20, U5 to U3, U6 to U4, U7 to U5, U8 to U6, U9 to U7, U10 to U8, U11 to U9
