File: Usb_Power.kicad_sch (KiCad schematic)
At the start: 18 parts, among them J2 USB_C_Receptacle_USB2.0_16P, U1 AMS1117-3.3, U2 USBLC6-2SC6

Commit message: Modified Power supplies, lost some sanity
Parts:
- removed U1: AMS1117-3.3, Package_TO_SOT_SMD:SOT-223-3_TabPin2, symbol Regulator_Linear:AMS1117-3.3
- added C32, C36: 1u, Capacitor_SMD:C_0603_1608Metric_Pad1.08x0.95mm_HandSolder, symbol Device:C
- added U22, U23: TLV1117-33, symbol Regulator_Linear:TLV1117-33
- C31: renamed from C1; value 47u -> 1u
- C35: renamed from C2; value 22u -> 1u
- renumbered C38 to C23, C39 to C24, C40 to C25, C41 to C26, C42 to C27, C43 to C28, C44 to C29, C45 to C30, C46 to C33, C47 to C34, J2 to J3, R1 to R6, R2 to R7, R3 to R8, U2 to U21
Connections:
- net +3.3V: now also U22.2 (VO)
- net +5V: now also C32.1, U22.3 (VI), U23.3 (VI)
- net GND: now also C32.2, C36.2, U22.1 (GND), U23.1 (GND)
- new net +3.3VA: C36.1, U23.2 (VO)
Other:
- note added: "3.3V reference (D+A)"
- note removed: "3.3V reference (TBD AP2114H-3.3) ???"
- moved on the sheet: C31, C35

Commit message: Minor fixes
Other:
- note added: "Either way we will have one single GND Polygon..."
- note removed: "Done on the MCU GND SIDE ONLY"
Changed lines of the file:
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@@
 	(rectangle
 		(start 13.97 124.46)
-		(end 92.71 152.4)
+		(end 92.71 153.67)
 		(stroke
 			(width 0.254)
@@
 		)
 	)
-	(text "Done on the MCU GND SIDE ONLY"
+	(text "Either way we will have one single GND Polygon..."
 		(exclude_from_sim no)
-		(at 49.53 144.018 0)
+		(at 53.34 148.336 0)
 		(effects
 			(font
-				(size 2.54 2.54)
-				(thickness 0.508)
-				(bold yes)
-				(color 255 0 0 1)
+				(size 1.778 1.778)
+				(thickness 0.254)
 			)
 		)
@@
 	)
 	(junction
-		(at 49.53 132.08)
+		(at 49.53 135.89)
 		(diameter 0)
 		(color 0 0 0 0)
@@
 	(wire
 		(pts
-			(xy 46.99 132.08) (xy 49.53 132.08)
+			(xy 46.99 135.89) (xy 49.53 135.89)
 		)
 		(stroke
@@
 	(wire
 		(pts
-			(xy 53.34 134.62) (xy 53.34 132.08)
+			(xy 53.34 138.43) (xy 53.34 135.89)
 		)
 		(stroke
@@
 	(wire
 		(pts
-			(xy 49.53 132.08) (xy 53.34 132.08)
+			(xy 49.53 135.89) (xy 53.34 135.89)
 		)
 		(stroke
@@
 	(wire
 		(pts
-			(xy 46.99 134.62) (xy 46.99 132.08)
+			(xy 46.99 138.43) (xy 46.99 135.89)
 		)
 		(stroke
@@
 	(symbol
 		(lib_id "power:PWR_FLAG")
-		(at 49.53 132.08 0)
+		(at 49.53 135.89 0)
 		(unit 1)
 		(body_style 1)
@@
 		(dnp no)
 		(property "Reference" "#FLG03"
-			(at 49.53 130.175 0)
+			(at 49.53 133.985 0)
 			(hide yes)
 			(show_name no)
@@
 		)
 		(property "Value" "PWR_FLAG"
-			(at 55.626 130.302 0)
+			(at 55.626 134.112 0)
 			(show_name no)
 			(do_not_autoplace no)
@@
 		)
 		(property "Footprint" ""
-			(at 49.53 132.08 0)
+			(at 49.53 135.89 0)
 			(hide yes)
 			(show_name no)
@@
 		)
 		(property "Datasheet" ""
-			(at 49.53 132.08 0)
+			(at 49.53 135.89 0)
 			(hide yes)
 			(show_name no)
@@
 		)
 		(property "Description" "Special symbol for telling ERC where power comes from"
-			(at 49.53 132.08 0)
+			(at 49.53 135.89 0)
 			(hide yes)
 			(show_name no)
@@
 	(symbol
 		(lib_id "power:GNDA")
-		(at 46.99 134.62 0)
+		(at 46.99 138.43 0)
 		(unit 1)
 		(body_style 1)
@@
 		(dnp no)
 		(property "Reference" "#PWR067"
-			(at 46.99 140.97 0)
+			(at 46.99 144.78 0)
 			(hide yes)
 			(show_name no)
@@
 		)
 		(property "Value" "GNDA"
-			(at 46.482 138.43 0)
+			(at 46.482 142.24 0)
 			(show_name no)
 			(do_not_autoplace no)
@@
 		)
 		(property "Footprint" ""
-			(at 46.99 134.62 0)
+			(at 46.99 138.43 0)
 			(hide yes)
 			(show_name no)
@@
 		)
 		(property "Datasheet" ""
-			(at 46.99 134.62 0)
+			(at 46.99 138.43 0)
 			(hide yes)
 			(show_name no)
@@
 		)
 		(property "Description" "Power symbol creates a global label with name \"GNDA\" , analog ground"
-			(at 46.99 134.62 0)
+			(at 46.99 138.43 0)
 			(hide yes)
 			(show_name no)
@@
 	(symbol
 		(lib_id "power:GNDD")
-		(at 53.34 134.62 0)
+		(at 53.34 138.43 0)
 		(unit 1)
 		(body_style 1)
@@
 		(dnp no)
 		(property "Reference" "#PWR069"
-			(at 53.34 140.97 0)
+			(at 53.34 144.78 0)
 			(hide yes)
 			(show_name no)
@@
 		)
 		(property "Value" "GND"
-			(at 53.848 138.43 0)
+			(at 53.848 142.24 0)
 			(show_name no)
 			(do_not_autoplace no)
@@
 		)
 		(property "Footprint" ""
-			(at 53.34 134.62 0)
+			(at 53.34 138.43 0)
 			(hide yes)
 			(show_name no)
@@
 		)
 		(property "Datasheet" ""
-			(at 53.34 134.62 0)
+			(at 53.34 138.43 0)
 			(hide yes)
 			(show_name no)
@@
 		)
 		(property "Description" "Power symbol creates a global label with name \"GNDD\" , digital ground"
-			(at 53.34 134.62 0)
+			(at 53.34 138.43 0)
 			(hide yes)
 			(show_name no)
