File: keyhalld-addon/keyhalld-addon.kicad_sch (KiCad schematic)
At the start: 0 parts

Commit message: move common libs to root; add fp to ldo
Parts:
- added U1: RP2350A, RPI:rpi_rp2350a_vias, symbol RPI_DB:Integrated_Circuits | Microcontrollers/RP-01HA9H-9K5E8T

Commit message: update addon board to minimal schematic
Parts:
- removed U1: RP2350A, RPI:rpi_rp2350a_vias, symbol RPI_DB:Integrated_Circuits | Microcontrollers/RP-01HA9H-9K5E8T
- added C1, C10, C2, C3, C4, C5, C6, C7, C8, C9: 100n, Capacitor_SMD:C_0603_1608Metric_Pad1.08x0.95mm_HandSolder, symbol Device:C
- added C11, C12: 1u, Capacitor_SMD:C_0603_1608Metric_Pad1.08x0.95mm_HandSolder, symbol Device:C
- added C13, C14: 4.7u, Capacitor_SMD:C_0603_1608Metric, symbol Device:C
- added C16, C17: 15p, Capacitor_SMD:C_0603_1608Metric_Pad1.08x0.95mm_HandSolder, symbol Device:C
- added J1: Conn_01x06_Pin, Connector_PinHeader_2.54mm:PinHeader_1x06_P2.54mm_Horizontal, symbol Connector:Conn_01x06_Pin
- added J2: Conn_01x04_Pin, Connector_Wire:SolderWire-0.127sqmm_1x04_P3.7mm_D0.48mm_OD1mm, symbol Connector:Conn_01x04_Pin
- added L1: 3.3uH, Inductor_SMD:L_Murata_DFE201610P, symbol Device:L
- added R1, R10, R11, R2, R3, R4, R8, R9: 10K, Resistor_SMD:R_0603_1608Metric_Pad0.98x0.95mm_HandSolder, symbol Device:R
- added R12: 1K, Resistor_SMD:R_0603_1608Metric_Pad0.98x0.95mm_HandSolder, symbol Device:R
- added SW1, SW2, SW3, SW4, SW5, SW6, SW7, SW8: SW_Push, Switch_Keyboard_Cherry_MX:SW_Cherry_MX_PCB_1.00u, symbol Switch:SW_Push
- added U1: TLV1117-33, Package_TO_SOT_SMD:SOT-223, symbol Regulator_Linear:TLV1117-33
- added U2: RP2350A, RPI:rpi_rp2350a_vias, symbol RPI_DB:Integrated_Circuits | Microcontrollers/RP-01HA9H-9K5E8T
- added U3: ER_OLEDM0.91_1x-I2C, Display:ER_OLEDM0.91_1x-I2C, symbol Display_Graphic:ER_OLEDM0.91_1x-I2C
- added Y1: 12MHz, Oscillator:Oscillator_SMD_Abracon_ASE-4Pin_3.2x2.5mm, symbol RPI_DB:Frequency_Timing | Crystals/RP-01G8X7-GS352B
Connections:
- new net: C17.2, R12.2, Y1.3
- new net: L1.2, U2.48 (VREG_LX)
- new net +1V1: C10.1, C13.1, C8.1, C9.1, L1.1, U2.23 (DVDD), U2.39 (DVDD), U2.50 (VREG_FB), U2.6 (DVDD)
- new net +3.3V: C1.1, C12.1, C14.1, C2.1, C3.1, C4.1, C5.1, C6.1, C7.1, J1.1 (Pin_1), R1.1, R10.1, R11.1, R2.1, R3.1, R4.1, R8.1, R9.1, U1.2 (VO), U2.1 (IOVDD), U2.11 (IOVDD), U2.20 (IOVDD), U2.30 (IOVDD), U2.38 (IOVDD), U2.44 (ADC_AVDD), U2.45 (IOVDD), U2.46 (VREG_AVDD), U2.49 (VREG_VIN), U2.53 (USB_OTP_VDD), U2.54 (QSPI_IOVDD), U3.2 (VCC)
- new net +5V: C11.1, J2.1 (Pin_1), U1.3 (VI)
- new net DBG_TX: J1.5 (Pin_5), U2.2 (GPIO0)
- new net GND: C1.2, C10.2, C11.2, C12.2, C13.2, C14.2, C16.1, C17.1, C2.2, C3.2, C4.2, C5.2, C6.2, C7.2, C8.2, C9.2, J1.6 (Pin_6), J2.4 (Pin_4), SW1.2, SW2.2, SW3.2, SW4.2, SW5.2, SW6.2, SW7.2, SW8.2, U1.1 (GND), U2.47 (VREG_PGND), U2.61 (GND), U3.1 (GND), Y1.2, Y1.4
- new net KEY1: R1.2, SW1.1, U2.12 (GPIO8)
- new net KEY2: R2.2, SW2.1, U2.13 (GPIO9)
- new net KEY3: R3.2, SW3.1, U2.14 (GPIO10)
- new net KEY4: R4.2, SW4.1, U2.15 (GPIO11)
- new net KEY5: R8.2, SW5.1, U2.16 (GPIO12)
- new net KEY6: R9.2, SW6.1, U2.17 (GPIO13)
- new net KEY7: R10.2, SW7.1, U2.18 (GPIO14)
- new net KEY8: R11.2, SW8.1, U2.19 (GPIO15)
- new net MAG_UART_RX: J2.3 (Pin_3), U2.8 (GPIO5)
- new net MAG_UART_TX: J2.2 (Pin_2), U2.7 (GPIO4)
- new net OLED_SCL: U2.10 (GPIO7), U3.3 (SCL)
- new net OLED_SDA: U2.9 (GPIO6), U3.4 (SDA)
- new net RUN: J1.4 (Pin_4), U2.26 (RUN)
- new net SWCLK: J1.2 (Pin_2), U2.24 (SWCLK)
- new net SWDIO: J1.3 (Pin_3), U2.25 (SWDIO)
- new net XIN: C16.2, U2.21 (XIN), Y1.1
- new net XOUT: R12.1, U2.22 (XOUT)
- no-connect marks 0 -> 25
Other:
- note added: "3.3V reference"
- note added: "Clocking"
- note added: "Debug header"
- note added: "Decoupling caps for DVDD"
- note added: "Decoupling caps for IOVDD"
- note added: "MX Switches array"
- note added: "MagSafe"
- note added: "Oleg"
- note added: "Power Decoupling"
- note added: "RPi Does not support SWO"
- title: (none) -> Expansion board for main keyhalld board

Commit message: add local fp for cherry mx mech switch
Parts:
- SW1, SW2, SW3, SW4, SW5, SW6, SW7, SW8: footprint Switch_Keyboard_Cherry_MX:SW_Cherry_MX_PCB_1.00u -> Library:SW_Cherry_MX_PCB_1.00u
Changed lines of the file:
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@@
 			)
 		)
-		(property "Footprint" "Switch_Keyboard_Cherry_MX:SW_Cherry_MX_PCB_1.00u"
+		(property "Footprint" "Library:SW_Cherry_MX_PCB_1.00u"
 			(at 147.32 95.25 0)
 			(hide yes)
@@
 			)
 		)
-		(property "Footprint" "Switch_Keyboard_Cherry_MX:SW_Cherry_MX_PCB_1.00u"
+		(property "Footprint" "Library:SW_Cherry_MX_PCB_1.00u"
 			(at 71.12 95.25 0)
 			(hide yes)
@@
 			)
 		)
-		(property "Footprint" "Switch_Keyboard_Cherry_MX:SW_Cherry_MX_PCB_1.00u"
+		(property "Footprint" "Library:SW_Cherry_MX_PCB_1.00u"
 			(at 121.92 69.85 0)
 			(hide yes)
@@
 			)
 		)
-		(property "Footprint" "Switch_Keyboard_Cherry_MX:SW_Cherry_MX_PCB_1.00u"
+		(property "Footprint" "Library:SW_Cherry_MX_PCB_1.00u"
 			(at 147.32 69.85 0)
 			(hide yes)
@@
 			)
 		)
-		(property "Footprint" "Switch_Keyboard_Cherry_MX:SW_Cherry_MX_PCB_1.00u"
+		(property "Footprint" "Library:SW_Cherry_MX_PCB_1.00u"
 			(at 96.52 95.25 0)
 			(hide yes)
@@
 			)
 		)
-		(property "Footprint" "Switch_Keyboard_Cherry_MX:SW_Cherry_MX_PCB_1.00u"
+		(property "Footprint" "Library:SW_Cherry_MX_PCB_1.00u"
 			(at 121.92 95.25 0)
 			(hide yes)
@@
 			)
 		)
-		(property "Footprint" "Switch_Keyboard_Cherry_MX:SW_Cherry_MX_PCB_1.00u"
+		(property "Footprint" "Library:SW_Cherry_MX_PCB_1.00u"
 			(at 71.12 69.85 0)
 			(hide yes)
@@
 			)
 		)
-		(property "Footprint" "Switch_Keyboard_Cherry_MX:SW_Cherry_MX_PCB_1.00u"
+		(property "Footprint" "Library:SW_Cherry_MX_PCB_1.00u"
 			(at 96.52 69.85 0)
 			(hide yes)

Commit message: fix some custom fp; change fp for mech keys to hotswap
Parts:
- SW1, SW2, SW3, SW4, SW5, SW6, SW7, SW8: footprint Library:SW_Cherry_MX_PCB_1.00u -> Library:SW_Hotswap_Kailh_MX_1.00u
Changed lines of the file:
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@@
 			)
 		)
-		(property "Footprint" "Library:SW_Cherry_MX_PCB_1.00u"
+		(property "Footprint" "Library:SW_Hotswap_Kailh_MX_1.00u"
 			(at 147.32 95.25 0)
 			(hide yes)
@@
 			)
 		)
-		(property "Footprint" "Library:SW_Cherry_MX_PCB_1.00u"
+		(property "Footprint" "Library:SW_Hotswap_Kailh_MX_1.00u"
 			(at 71.12 95.25 0)
 			(hide yes)
@@
 			)
 		)
-		(property "Footprint" "Library:SW_Cherry_MX_PCB_1.00u"
+		(property "Footprint" "Library:SW_Hotswap_Kailh_MX_1.00u"
 			(at 121.92 69.85 0)
 			(hide yes)
@@
 			)
 		)
-		(property "Footprint" "Library:SW_Cherry_MX_PCB_1.00u"
+		(property "Footprint" "Library:SW_Hotswap_Kailh_MX_1.00u"
 			(at 147.32 69.85 0)
 			(hide yes)
@@
 			)
 		)
-		(property "Footprint" "Library:SW_Cherry_MX_PCB_1.00u"
+		(property "Footprint" "Library:SW_Hotswap_Kailh_MX_1.00u"
 			(at 96.52 95.25 0)
 			(hide yes)
@@
 			)
 		)
-		(property "Footprint" "Library:SW_Cherry_MX_PCB_1.00u"
+		(property "Footprint" "Library:SW_Hotswap_Kailh_MX_1.00u"
 			(at 121.92 95.25 0)
 			(hide yes)
@@
 			)
 		)
-		(property "Footprint" "Library:SW_Cherry_MX_PCB_1.00u"
+		(property "Footprint" "Library:SW_Hotswap_Kailh_MX_1.00u"
 			(at 71.12 69.85 0)
 			(hide yes)
@@
 			)
 		)
-		(property "Footprint" "Library:SW_Cherry_MX_PCB_1.00u"
+		(property "Footprint" "Library:SW_Hotswap_Kailh_MX_1.00u"
 			(at 96.52 69.85 0)
 			(hide yes)

Commit message: add option for usb connection to addon board; initial addon pcb layout
Parts:
- added J2: USB_C_Receptacle_USB2.0_16P, Connector_USB:USB_C_Receptacle_GCT_USB4105-xx-A_16P_TopMnt_Horizontal, symbol Connector:USB_C_Receptacle_USB2.0_16P
- added R12, R13: 5K1, Resistor_SMD:R_0603_1608Metric_Pad0.98x0.95mm_HandSolder, symbol Device:R
- added R14: 1.5K, Resistor_SMD:R_0603_1608Metric_Pad0.98x0.95mm_HandSolder, symbol Device:R
- added R5, R6: 22R, Resistor_SMD:R_0603_1608Metric_Pad0.98x0.95mm_HandSolder, symbol Device:R
- added U3: USBLC6-2SC6, Package_TO_SOT_SMD:SOT-23-6, symbol Power_Protection:USBLC6-2SC6
- renumbered C16 to C15, C17 to C16, J2 to J3, R11 to R10, R12 to R11, R8 to R7, R9 to R8, R10 to R9, U3 to U4
Connections:
- net +3.3V: now also R14.2
- net +5V: now also J2.A4 (VBUS), J2.A9 (VBUS), J2.B4 (VBUS), J2.B9 (VBUS), U3.5 (VBUS)
- net GND: now also J2.A1 (GND), J2.A12 (GND), J2.B1 (GND), J2.B12 (GND), J2.SH (SHIELD), R12.2, R13.1, U3.2 (GND)
- net at U2.51 (USB_DM): now also R6.2
- net at U2.52 (USB_DP): now also R5.1
- new net: J2.A5 (CC1), R12.1
- new net: J2.B5 (CC2), R13.2
- new net CONN_D+: J2.A6 (D+), J2.B6 (D+), R14.1, U3.3 (I/O2)
- new net CONN_D-: J2.A7 (D-), J2.B7 (D-), U3.1 (I/O1)
- new net D+: R5.2, U3.4 (I/O2)
- new net D-: R6.1, U3.6 (I/O1)
Other:
- note added: "USB Connector & ESD Protection"

Commit message: small adjustments
Other:
- note added: "Optional part for this board Needed if planned to be used independedly (in that case board will need separate FW)"
Changed lines of the file:
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@@
+		)
+	)
+	(text "Optional part for this board\nNeeded if planned to be used independedly\n(in that case board will need separate FW)"
+		(exclude_from_sim no)
+		(at 134.112 170.434 0)
+		(effects
+			(font
+				(size 1.524 1.524)
+				(thickness 0.508)
+				(bold yes)
+			)
+			(justify right)
 		)
 	)

Commit message: save the work
Parts:
- added R1, R2, R3, R4, R5, R6, R7: 10K, Resistor_SMD:R_0603_1608Metric_Pad0.98x0.95mm_HandSolder, symbol Device:R
- added R14, R20, R21: 4K7, Resistor_SMD:R_0603_1608Metric_Pad0.98x0.95mm_HandSolder, symbol Device:R
- added S1: RKJXT1F42001, Library:XDCR_RKJXT1F42001, symbol RKJXT1F42001:RKJXT1F42001
- added SW10: RST, Button_Switch_SMD:SW_Tactile_SPST_NO_Straight_CK_PTS636Sx25SMTRLFS, symbol Switch:SW_Push
- added SW9: BOOT, Button_Switch_SMD:SW_Tactile_SPST_NO_Straight_CK_PTS636Sx25SMTRLFS, symbol Switch:SW_Push
- renumbered R3 to R10, R4 to R11, R5 to R12, R6 to R13, R7 to R15, R8 to R16, R9 to R17, R10 to R18, R11 to R19, R12 to R22, R13 to R23, R14 to R24, R1 to R8, R2 to R9
Connections:
- net +3.3V: now also R1.1, R2.2, R20.2, R21.1, R3.1, R4.2, R5.1, R6.2, R7.1
- net GND: now also U2.59 (QSPI_SD1), S1.COM, S1.EN_COM, S1.GND, SW10.2, SW9.2
- net OLED_SCL: now also R21.2
- net OLED_SDA: now also R20.1
- net RUN: now also SW10.1
- net EN_A: now reaches U2.31 (GPIO19)
- net EN_A: now also R3.2, S1.EN_A
- net EN_B: now reaches U2.32 (GPIO20)
- net EN_B: now also R4.1, S1.EN_B
- net EN_S_P: now reaches U2.33 (GPIO21)
- net EN_S_P: now also R5.2, S1.P (PUSH)
- net EN_S_A: now reaches U2.34 (GPIO22)
- net EN_S_A: now also R1.2, S1.A
- net EN_S_B: now reaches U2.35 (GPIO23)
- net EN_S_B: now also R2.1, S1.B
- net EN_S_C: now reaches U2.36 (GPIO24)
- net EN_S_C: now also R6.1, S1.C
- net EN_S_D: now reaches U2.37 (GPIO25)
- net EN_S_D: now also R7.2, S1.D
- net at U2.60 (QSPI_~{SS}): now also R14.1
- new net BOOT: R14.2, SW9.1
- no-connect marks 25 -> 16
Other:
- note added: "Automobile Encoder"
- note added: "Boot/Reset"

Commit message: maybe last schematic changes; pcb new layout
Parts:
- added D1, D2: D, Diode_SMD:D_SOD-323, symbol Device:D
- added H1, H2, H3, H4: MountingHole_Pad, MountingHole:MountingHole_2.2mm_M2_DIN965_Pad, symbol Mechanical:MountingHole_Pad
Connections:
- net +5V: now also D1.2 (A), D2.1 (K); no longer J2.A4 (VBUS), J2.A9 (VBUS), J2.B4 (VBUS), J2.B9 (VBUS), J3.1 (Pin_1)
- net GND: now also H1.1, H2.1, H3.1, H4.1
- new net: D2.2 (A), J2.A4 (VBUS), J2.A9 (VBUS), J2.B4 (VBUS), J2.B9 (VBUS)
- new net: D1.1 (K), J3.1 (Pin_1)
Other:
- note added: "Mounting Holes"
