File: keyhalld-addon/ws_leds.kicad_sch (KiCad schematic)
At the start: 8 parts

Commit message: Super changes; FInal!
Parts:
- added D3: WS2812B-2020 STATUS, LED_SMD:LED_WS2812B-2020_PLCC4_2.0x2.0mm, symbol LED:WS2812B-2020
- renumbered D9 to D10, D10 to D11, D3 to D4, D4 to D5, D5 to D6, D6 to D7, D7 to D8, D8 to D9
Connections:
- net +5V: now also D3.4 (VDD)
- net GND: now also D3.2 (VSS)
- net WS_IN: no longer names the net of D4.3 (DIN)
- net WS_IN: now also D3.1 (DOUT)
- new net WS_LED: D3.3 (DIN)
Other:
- moved on the sheet: D10, D11, D4, D5, D6, D7, D8, D9

Commit message: routed pcb for addon board
Parts:
- added C17, C18, C19, C20, C21, C22, C23, C24, C25: 100n, Capacitor_SMD:C_0603_1608Metric, symbol Device:C
- D3: value WS2812B-2020 STATUS -> STATUS
Connections:
- net +5V: now also C17.2, C18.2, C19.2, C20.2, C21.2, C22.2, C23.2, C24.2, C25.2
- net GND: now also C17.1, C18.1, C19.1, C20.1, C21.1, C22.1, C23.1, C24.1, C25.1
Other:
- moved on the sheet: D10, D11, D8, D9
