File: keyhalld-addon/keyhalld-addon.kicad_pcb (KiCad board)
At the start: 4 copper layers, 140 x 40 mm, 85 parts, among them J1 Conn_01x06_Pin, J2 USB_C_Receptacle_USB2.0_16P, J3 Conn_01x04_Pin, SW1 SW_Push, SW10 RST, SW2 SW_Push, SW3 SW_Push, SW4 SW_Push, SW5 SW_Push, SW6 SW_Push, SW7 SW_Push, SW8 SW_Push, SW9 BOOT, U1 TLV1117-33, U2 RP2350A, U3 USBLC6-2SC6, U4 ER_OLEDM0.91_1x-I2C, Y1 12MHz

Commit message: littpe powerline tweaks
Routing:
- net +3.3V: track 244.3 -> 255.4 mm
- net Net-(D8-DOUT): track 26.7 -> 25.8 mm
- net Net-(D7-DOUT): track 76.6 -> 77.2 mm

Commit message: adjusut usb and power routuing
Routing:
- net +3.3V: track 255.4 -> 253.1 mm, vias 15 -> 16
- net +1V1: track 39.6 -> 40.4 mm
- net D+: track 17.9 -> 17.2 mm
- net GND: vias 278 -> 282

Commit message: remove via litter
Routing:
- net +3.3V: track 253.1 -> 321.3 mm
- net GND: vias 282 -> 99
- removed copper zone on In1.Cu, net +3.3V
