File: keyhalld/Usb_Power.kicad_sch (KiCad schematic)
At the start: 21 parts, among them J3 USB_C_Receptacle_USB2.0_16P, U21 USBLC6-2SC6, U22 TLV1117-33, U23 TLV1117-33

Commit message: move common libs to root; add fp to ldo
Parts:
- U22, U23: footprint (none) -> Package_TO_SOT_SMD:SOT-223
Changed lines of the file:
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@@
 			)
 		)
-		(property "Footprint" ""
+		(property "Footprint" "Package_TO_SOT_SMD:SOT-223"
 			(at 116.84 78.74 0)
 			(hide yes)
@@
 			)
 		)
-		(property "Footprint" ""
+		(property "Footprint" "Package_TO_SOT_SMD:SOT-223"
 			(at 116.84 104.14 0)
 			(hide yes)

Commit message: Started PCB Implementation
Parts:
- renumbered C23 to C25, C24 to C26, C25 to C27, C26 to C28, C27 to C29, C28 to C30, C29 to C31, C30 to C32, C31 to C35, C35 to C36, C32 to C37, C36 to C38, U22 to U21, U21 to U22

Commit message: Sch refactor, power part done (for MCU)
Parts:
- removed C26: 100n, Capacitor_SMD:C_0603_1608Metric_Pad1.08x0.95mm_HandSolder, symbol Device:C
- added C31, C32: 100n, Capacitor_SMD:C_0603_1608Metric_Pad1.08x0.95mm_HandSolder, symbol Device:C
- renumbered C27 to C26, C28 to C27, C29 to C28, C30 to C29, C31 to C30, C32 to C33, C33 to C34, C34 to C35, C35 to C36, C36 to C37, C37 to C38, C38 to C39
Connections:
- net +3.3V: now also C31.1
- net +3.3VA: now also C32.1
- net GND: now also C31.2, C32.2
Other:
- moved on the sheet: C25, C26, C27, C28, C29, C30, C33, C34, C35
