File: keyhalld/hallswitches.kicad_sch (KiCad schematic)
At the start: 54 parts, among them SW1 HallSwitch, SW10 HallSwitch, SW11 HallSwitch, SW12 HallSwitch, SW13 HallSwitch, SW14 HallSwitch, SW15 HallSwitch, SW16 HallSwitch, SW17 HallSwitch, SW18 HallSwitch, SW2 HallSwitch, SW3 HallSwitch, SW4 HallSwitch, SW5 HallSwitch, SW6 HallSwitch, SW7 HallSwitch, SW8 HallSwitch, SW9 HallSwitch, U10 DRV5055A4xDBZxQ1, U11 DRV5055A4xDBZxQ1, U12 DRV5055A4xDBZxQ1, U13 DRV5055A4xDBZxQ1, U14 DRV5055A4xDBZxQ1, U15 DRV5055A4xDBZxQ1, U16 DRV5055A4xDBZxQ1, U17 DRV5055A4xDBZxQ1, U18 DRV5055A4xDBZxQ1, U19 DRV5055A4xDBZxQ1, U20 DRV5055A4xDBZxQ1, U3 DRV5055A4xDBZxQ1, U4 DRV5055A4xDBZxQ1, U5 DRV5055A4xDBZxQ1, U6 DRV5055A4xDBZxQ1, U7 DRV5055A4xDBZxQ1, U8 DRV5055A4xDBZxQ1, U9 DRV5055A4xDBZxQ1

Commit message: move common libs to root; add fp to ldo
Parts:
- SW1, SW10, SW11, SW12, SW13, SW14, SW15, SW16, SW17, SW18, SW2, SW3, SW4, SW5, SW6, SW7, SW8, SW9: footprint Custom:Custom_MX_PCB_1.00u -> Library:Custom_MX_PCB_1.00u
Changed lines of the file:
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@@
 			)
 		)
-		(property "Footprint" "Custom:Custom_MX_PCB_1.00u"
+		(property "Footprint" "Library:Custom_MX_PCB_1.00u"
 			(at 26.67 36.83 0)
 			(hide yes)
@@
 			)
 		)
-		(property "Footprint" "Custom:Custom_MX_PCB_1.00u"
+		(property "Footprint" "Library:Custom_MX_PCB_1.00u"
 			(at 80.01 36.83 0)
 			(hide yes)
@@
 			)
 		)
-		(property "Footprint" "Custom:Custom_MX_PCB_1.00u"
+		(property "Footprint" "Library:Custom_MX_PCB_1.00u"
 			(at 53.34 132.08 0)
 			(hide yes)
@@
 			)
 		)
-		(property "Footprint" "Custom:Custom_MX_PCB_1.00u"
+		(property "Footprint" "Library:Custom_MX_PCB_1.00u"
 			(at 106.68 36.83 0)
 			(hide yes)
@@
 			)
 		)
-		(property "Footprint" "Custom:Custom_MX_PCB_1.00u"
+		(property "Footprint" "Library:Custom_MX_PCB_1.00u"
 			(at 133.35 36.83 0)
 			(hide yes)
@@
 			)
 		)
-		(property "Footprint" "Custom:Custom_MX_PCB_1.00u"
+		(property "Footprint" "Library:Custom_MX_PCB_1.00u"
 			(at 186.69 36.83 0)
 			(hide yes)
@@
 			)
 		)
-		(property "Footprint" "Custom:Custom_MX_PCB_1.00u"
+		(property "Footprint" "Library:Custom_MX_PCB_1.00u"
 			(at 26.67 132.08 0)
 			(hide yes)
@@
 			)
 		)
-		(property "Footprint" "Custom:Custom_MX_PCB_1.00u"
+		(property "Footprint" "Library:Custom_MX_PCB_1.00u"
 			(at 186.69 85.09 0)
 			(hide yes)
@@
 			)
 		)
-		(property "Footprint" "Custom:Custom_MX_PCB_1.00u"
+		(property "Footprint" "Library:Custom_MX_PCB_1.00u"
 			(at 213.36 36.83 0)
 			(hide yes)
@@
 			)
 		)
-		(property "Footprint" "Custom:Custom_MX_PCB_1.00u"
+		(property "Footprint" "Library:Custom_MX_PCB_1.00u"
 			(at 26.67 85.09 0)
 			(hide yes)
@@
 			)
 		)
-		(property "Footprint" "Custom:Custom_MX_PCB_1.00u"
+		(property "Footprint" "Library:Custom_MX_PCB_1.00u"
 			(at 106.68 85.09 0)
 			(hide yes)
@@
 			)
 		)
-		(property "Footprint" "Custom:Custom_MX_PCB_1.00u"
+		(property "Footprint" "Library:Custom_MX_PCB_1.00u"
 			(at 213.36 85.09 0)
 			(hide yes)
@@
 			)
 		)
-		(property "Footprint" "Custom:Custom_MX_PCB_1.00u"
+		(property "Footprint" "Library:Custom_MX_PCB_1.00u"
 			(at 53.34 36.83 0)
 			(hide yes)
@@
 			)
 		)
-		(property "Footprint" "Custom:Custom_MX_PCB_1.00u"
+		(property "Footprint" "Library:Custom_MX_PCB_1.00u"
 			(at 53.34 85.09 0)
 			(hide yes)
@@
 			)
 		)
-		(property "Footprint" "Custom:Custom_MX_PCB_1.00u"
+		(property "Footprint" "Library:Custom_MX_PCB_1.00u"
 			(at 133.35 85.09 0)
 			(hide yes)
@@
 			)
 		)
-		(property "Footprint" "Custom:Custom_MX_PCB_1.00u"
+		(property "Footprint" "Library:Custom_MX_PCB_1.00u"
 			(at 160.02 36.83 0)
 			(hide yes)
@@
 			)
 		)
-		(property "Footprint" "Custom:Custom_MX_PCB_1.00u"
+		(property "Footprint" "Library:Custom_MX_PCB_1.00u"
 			(at 160.02 85.09 0)
 			(hide yes)
@@
 			)
 		)
-		(property "Footprint" "Custom:Custom_MX_PCB_1.00u"
+		(property "Footprint" "Library:Custom_MX_PCB_1.00u"
 			(at 80.01 85.09 0)
 			(hide yes)

Commit message: Schematic done for Motherboard
Changed lines of the file:
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@@
 	(text "Hall Sensor footprint should be centered underneath switch!!!"
 		(exclude_from_sim no)
-		(at 188.214 157.988 0)
+		(at 175.26 155.194 0)
 		(effects
 			(font

Commit message: Started PCB Implementation
Parts:
- renumbered C8 to C10, C13 to C12, C15 to C13, C17 to C14, C19 to C15, C21 to C16, C6 to C17, C9 to C18, C12 to C19, C14 to C20, C16 to C21, C18 to C22, C20 to C23, C22 to C24, C10 to C8, C5 to C9, SW13 to SW10, SW15 to SW11, SW17 to SW12, SW2 to SW13, SW5 to SW14, SW8 to SW15, SW10 to SW16, SW12 to SW17, SW14 to SW18, SW16 to SW19, SW18 to SW20, SW6 to SW4, SW1 to SW5, SW4 to SW6, SW9 to SW8, SW11 to SW9, U15 to U10, U17 to U11, U19 to U12, U4 to U13, U7 to U14, U10 to U15, U12 to U16, U14 to U17, U16 to U18, U18 to U19, U5 to U3, U8 to U4, U3 to U5, U9 to U7, U11 to U8, U13 to U9
Other:
- note added: "Dedicated switches"
- moved on the sheet: C10, C11, C12, C13, C14, C15, C16, C17, C18, C19, C20, C21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
