File: keyhalld/keyhalld.kicad_sch (KiCad schematic)
At the start: 28 parts, among them J1 Conn_01x06_Pin, J2 Conn_01x04_Pin, SW1 RESET, SW2 USB_BOOT, U1 RP2350A, U2 CD74HC4067M, Y1 12MHz

Commit message: Mega keyboard TBD need to validate
Parts:
- removed J1: Conn_01x06_Pin, Connector_PinHeader_2.54mm:PinHeader_1x06_P2.54mm_Horizontal, symbol Connector:Conn_01x06_Pin
- added D2: D_Schottky, symbol Device:D_Schottky
- added J1: Conn_01x05_Pin, Connector_PinHeader_2.54mm:PinHeader_1x05_P2.54mm_Horizontal, symbol Connector:Conn_01x05_Pin
Connections:
- net DBG_TX: now also J1.4 (Pin_4)
- net GND: now also J1.5 (Pin_5)
- net RUN: now also J1.3 (Pin_3)
- net SWCLK: now also J1.2 (Pin_2)
- net SWDIO: now also J1.1 (Pin_1)
