File: keyhalld/keyhalld.kicad_pcb (KiCad board)
At the start: 4 copper layers, 261 x 71 mm, 104 parts, among them J1 Conn_01x06_Pin, J2 Conn_01x04_Pin, J3 USB_C_Receptacle_USB2.0_16P, SW1 RESET, SW10 HallSwitch, SW11 HallSwitch, SW12 HallSwitch, SW13 HallSwitch, SW14 HallSwitch, SW15 HallSwitch, SW16 HallSwitch, SW17 HallSwitch, SW18 HallSwitch, SW19 HallSwitch, SW2 USB_BOOT, SW20 HallSwitch, SW3 HallSwitch, SW4 HallSwitch, SW5 HallSwitch, SW6 HallSwitch, SW7 HallSwitch, SW8 HallSwitch, SW9 HallSwitch, U1 RP2350A, U10 DRV5055A4xDBZxQ1, U11 DRV5055A4xDBZxQ1, U12 DRV5055A4xDBZxQ1, U13 DRV5055A4xDBZxQ1, U14 DRV5055A4xDBZxQ1, U15 DRV5055A4xDBZxQ1, U16 DRV5055A4xDBZxQ1, U17 DRV5055A4xDBZxQ1, U18 DRV5055A4xDBZxQ1, U19 DRV5055A4xDBZxQ1, U2 CD74HC4067M, U20 DRV5055A4xDBZxQ1, U21 TLV1117-33, U22 USBLC6-2SC6, U23 TLV1117-33, U3 DRV5055A4xDBZxQ1, U4 DRV5055A4xDBZxQ1, U5 DRV5055A4xDBZxQ1, U6 DRV5055A4xDBZxQ1, U7 DRV5055A4xDBZxQ1, U8 DRV5055A4xDBZxQ1, U9 DRV5055A4xDBZxQ1, Y1 12MHz

Commit message: Mega keyboard TBD need to validate
Parts:
- J1: value Conn_01x06_Pin -> Conn_01x05_Pin; footprint Connector_PinHeader_2.54mm:PinHeader_1x06_P2.54mm_Horizontal -> Connector_PinHeader_2.54mm:PinHeader_1x05_P2.54mm_Horizontal
- moved SW1 31.7 mm to (184.5, 114.5), turned to 0 degrees
- moved SW2 31.7 mm to (184.5, 119.5), turned to 0 degrees
- moved C37 2.80 mm to (164.0, 78.5)
- moved J1 2.42 mm to (171.8, 114.5)
- moved C36 1.35 mm to (169.8, 78.5)
- moved R1 1.11 mm to (176.2, 87.0), turned to 0 degrees
- moved C38 1.03 mm to (184.0, 72.5)
- moved C39 1.03 mm to (184.0, 76.5)
- moved C5 0.35 mm to (166.0, 104.6)
- moved J2 0.25 mm to (147.8, 92.4)
Connections:
- J1 pad 1: +3.3V -> SWDIO
- J1 pad 2: SWDIO -> SWCLK
- J1 pad 3: SWCLK -> RUN
- J1 pad 4: RUN -> DBG_TX
- J1 pad 5: DBG_TX -> GND
- U21 pad 4: (no net) -> +3.3V
- U23 pad 4: (no net) -> +3.3VA
Routing:
- net +3.3VA: track 98.3 -> 593.7 mm, vias 0 -> 26
- net Net-(U1-GPIO23): track 0.00 -> 128.5 mm
- net Net-(U1-GPIO22): track 0.00 -> 128.1 mm
- net Net-(U1-GPIO24): track 0.00 -> 117.5 mm
- net Net-(U1-GPIO25): track 0.00 -> 117.2 mm
- net Net-(U1-GPIO26_ADC0): track 0.00 -> 115.0 mm, vias 0 -> 2
- net GND: track 109.4 -> 195.4 mm, vias 6 -> 33
- net +3.3V: track 53.7 -> 103.7 mm, vias 5 -> 13
- net Net-(R5-Pad1): track 0.00 -> 49.4 mm, vias 0 -> 2
- net A1: track 0.00 -> 44.3 mm
- net +5V: track 65.8 -> 98.4 mm, vias 0 -> 1
- net RUN: track 6.68 -> 38.8 mm, vias 2 -> 1
- net A0: track 0.00 -> 26.5 mm
- net +1V1: track 22.7 -> 47.0 mm, vias 6 -> 7
- net MAG_UART_RX: track 0.00 -> 20.9 mm, vias 0 -> 2
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- added copper zone on In1.Cu, net GND

Commit message: Need2think about the Hall sensors + vias
Routing:
- net +3.3VA: track 593.7 -> 632.2 mm, vias 26 -> 27
